Commit message: Modify model/humanoid.urdf modified left shoulder origin pos

File: model/humanoid.urdf (robot description, URDF)
Before this commit: robot KHR1HV, 25 links, 24 joints
Joints:
- joint shoulder_left_pitch: origin xyz=0 0.15 0.0 rpy=0 0 0 -> xyz=0 0.055 0.0 rpy=0 0 0

Commit message: Modify urdf_file left leg is strange

File: model/humanoid.urdf (robot description, URDF)
Before this commit: robot KHR1HV, 25 links, 24 joints
Joints:
- joint hip_left_yaw: origin xyz=-0.1 0.02 -0.065 rpy=0 0 0 -> xyz=-0.025 0.02 -0.065 rpy=0 0 0
